Commit message: Add full 3D differential car project code, resolve gitignore conflict

File: src/car_description/urdf/car.gazebo.xacro (robot description, xacro)
@@ -106,77 +106,74 @@
   <!-- ============================================================-->
   <!-- IMU 仿真传感器 -->
-  <gazebo reference="imu_link">
-    <sensor name="imu_sensor" type="imu">
-      <always_on>true</always_on>
-      <update_rate>100</update_rate>
-      <visualize>false</visualize>
-      <body>imu_link</body>
-      <plugin filename="libgazebo_ros_imu_sensor.so" name="imu_plugin">
-        <ros>
-          <namespace>/</namespace>
-          <!-- 改为标准ROS2 IMU话题 imu/data -->
-          <remapping>~/out:=imu/data</remapping>
-        </ros>
-        <!-- 地面小车：以自身安装姿态为初始参考 -->
-        <initial_orientation_as_reference>true</initial_orientation_as_reference>
-        <!--描述 IMU姿态数据噪声可信度，管定位滤波-->
-        <orientation_covariance>1e-6 0 0  0 1e-6 0  0 0 1e-6</orientation_covariance>
-      </plugin>
-      <imu>
-        <angular_velocity>
-          <x>
-            <noise type="gaussian">
-              <mean>0.0</mean>
-              <stddev>2e-4</stddev>
-              <bias_mean>0.0000075</bias_mean>
-              <bias_stddev>0.0000008</bias_stddev>
-            </noise>
-          </x>
-          <y>
-            <noise type="gaussian">
-              <mean>0.0</mean>
-              <stddev>2e-4</stddev>
-              <bias_mean>0.0000075</bias_mean>
-              <bias_stddev>0.0000008</bias_stddev>
-            </noise>
-          </y>
-          <z>
-            <noise type="gaussian">
-              <mean>0.0</mean>
-              <stddev>2e-4</stddev>
-              <bias_mean>0.0000075</bias_mean>
-              <bias_stddev>0.0000008</bias_stddev>
-            </noise>
-          </z>
-        </angular_velocity>
-        <linear_acceleration>
-          <x>
-            <noise type="gaussian">
-              <mean>0.0</mean>
-              <stddev>1.7e-2</stddev>
-              <bias_mean>0.1</bias_mean>
-              <bias_stddev>0.001</bias_stddev>
-            </noise>
-          </x>
-          <y>
-            <noise type="gaussian">
-              <mean>0.0</mean>
-              <stddev>1.7e-2</stddev>
-              <bias_mean>0.1</bias_mean>
-              <bias_stddev>0.001</bias_stddev>
-            </noise>
-          </y>
-          <z>
-            <noise type="gaussian">
-              <mean>0.0</mean>
-              <stddev>1.7e-2</stddev>
-              <bias_mean>0.1</bias_mean>
-              <bias_stddev>0.001</bias_stddev>
-            </noise>
-          </z>
-        </linear_acceleration>
-      </imu>
-    </sensor>
-  </gazebo>
+  <gazebo reference="base_link">
+      <sensor name="imu_sensor" type="imu">
+        <always_on>true</always_on>
+        <update_rate>100</update_rate>
+        <visualize>false</visualize>
+        <plugin filename="libgazebo_ros_imu_sensor.so" name="imu_plugin">
+          <ros>
+            <namespace>/</namespace>
+            <remapping>~/out:=imu/data</remapping>
+          </ros>
+          <initial_orientation_as_reference>true</initial_orientation_as_reference>
+          <orientation_covariance>1e-6 0 0  0 1e-6 0  0 0 1e-6</orientation_covariance>
+          <frame_name>base_link</frame_name>
+        </plugin>
+        <imu>
+          <angular_velocity>
+            <x>
+              <noise type="gaussian">
+                <mean>0.0</mean>
+                <stddev>2e-4</stddev>
+                <bias_mean>0.0000075</bias_mean>
+                <bias_stddev>0.0000008</bias_stddev>
+              </noise>
+            </x>
+            <y>
+              <noise type="gaussian">
+                <mean>0.0</mean>
+                <stddev>2e-4</stddev>
+                <bias_mean>0.0000075</bias_mean>
+                <bias_stddev>0.0000008</bias_stddev>
+              </noise>
+            </y>
+            <z>
+              <noise type="gaussian">
+                <mean>0.0</mean>
+                <stddev>2e-4</stddev>
+                <bias_mean>0.0000075</bias_mean>
+                <bias_stddev>0.0000008</bias_stddev>
+              </noise>
+            </z>
+          </angular_velocity>
+          <linear_acceleration>
+            <x>
+              <noise type="gaussian">
+                <mean>0.0</mean>
+                <stddev>1.7e-2</stddev>
+                <bias_mean>0.1</bias_mean>
+                <bias_stddev>0.001</bias_stddev>
+              </noise>
+            </x>
+            <y>
+              <noise type="gaussian">
+                <mean>0.0</mean>
+                <stddev>1.7e-2</stddev>
+                <bias_mean>0.1</bias_mean>
+                <bias_stddev>0.001</bias_stddev>
+              </noise>
+            </y>
+            <z>
+              <noise type="gaussian">
+                <mean>0.0</mean>
+                <stddev>1.7e-2</stddev>
+                <bias_mean>0.1</bias_mean>
+                <bias_stddev>0.001</bias_stddev>
+              </noise>
+            </z>
+          </linear_acceleration>
+        </imu>
+      </sensor>
+    </gazebo>
   <!-- ============================================================-->
   <!-- 激光雷达 仿真插件 -->
@@ -184,5 +181,5 @@
     <sensor name="laser_sensor" type="ray">
       <always_on>true</always_on>
-      <visualize>false</visualize>
+      <visualize>true</visualize>
       <!-- 刷新频率改为10Hz，满足导航/SLAM需求 -->
       <update_rate>10</update_rate>
@@ -212,4 +209,5 @@
       <plugin name="laserscan" filename="libgazebo_ros_ray_sensor.so">
         <ros>
+          <argument>--ros-args -p use_sim_time:=true</argument>
           <remapping>~/out:=scan</remapping>
         </ros>
@@ -231,6 +229,6 @@
       <horizontal_fov>1.047</horizontal_fov>
       <image>
-        <width>640</width>
-        <height>480</height>
+        <width>320</width>
+        <height>240</height>
         <format>R8G8B8</format>
       </image>
@@ -249,16 +247,15 @@
     </camera>
     <!-- ROS2 通用相机插件（同时支持RGB+深度） -->
-        <plugin name="gazebo_ros_camera" filename="libgazebo_ros_camera.so">
+    <plugin name="gazebo_ros_camera" filename="libgazebo_ros_camera.so">
       <ros>
-        <!-- 关键：设置命名空间，统一话题前缀 -->
-        <remapping>~/image_raw:=image_raw</remapping>
-        <remapping>~/depth_image:=depth/image_raw</remapping>
-        <remapping>~/camera_info:=camera_info</remapping>
-      </ros>
+        <remapping>image_raw:=/depth_camera/image_raw</remapping>
+        <remapping>depth/image_raw:=/depth_camera/depth/image_raw</remapping>
+        <remapping>camera_info:=/depth_camera/camera_info</remapping>
+        <remapping>points:=/depth_camera/points</remapping> </ros>
       <frame_name>camera_color_optical_frame</frame_name>
       <depth>true</depth>
     </plugin>
   </sensor>
-</gazebo>
+ </gazebo>
 </xacro:macro>
 </robot>

File: src/car_description/urdf/car_base.urdf.xacro (robot description, xacro)
@@ -78,13 +78,5 @@
   </link>
   <!-- imu link -->
-  <link name="imu_link">
-    <visual>
-      <origin xyz="0 0 0.0" rpy="0 0 0"/>
-      <geometry>
-            <box size="0.02 0.02 0.02"/>
-      </geometry>
-    </visual>
-    <xacro:imu_physics />
-  </link>
+  <link name="imu_link"/>
   <!-- 深度相机 link -->
   <link name="depth_camera_link">
@@ -150,5 +142,5 @@
       <parent link="base_link" />
       <child link="imu_link" />
-      <origin xyz="0 0 0" />
+      <origin xyz="0 0 0" rpy="0 0 0" />
   </joint>
   <!-- 深度相机 固定关节，安装在车头最前端 -->
